File: pcb-v2/riser-v2.brd (EAGLE design)
At the start: 133.5 x 21.3 mm, 36 parts, among them IC1 SI53152-A01AGM, IC2 TPS51386RJNR, J1 MDT350M01001VTEXT, J2 MDT350M01001VTEXT, J3 PCI-E-X4, J4 0022053031, T1 2N7002, Y1 ECS-327KE-TR

Commit message: Mark DNP in EAGLE files too
Parts:
- C5: value 0.1uF -> DNP
Changed lines of the file:
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@@
 <attribute name="VALUE" x="6.635" y="16.405" size="1.27" layer="27" rot="R180"/>
 </element>
-<element name="C5" library="rcl" package="C0402" value="0.1uF" x="83" y="20" smashed="yes" rot="R270">
+<element name="C5" library="rcl" package="C0402" value="DNP" x="83" y="20" smashed="yes" rot="R270">
 <attribute name="NAME" x="85.3" y="12.5" size="1" layer="25" font="vector" ratio="16" rot="R270"/>
 <attribute name="VALUE" x="81.095" y="20.635" size="1.27" layer="27" rot="R270"/>
